Commit message: feat: Configure steering system hardware parameters, joint limits, and velocity state interface.

File: description/urdf/system_steering.urdf.xacro (robot description, xacro)
@@ -23,5 +23,6 @@
     <origin xyz="0.2 0 0" rpy="0 0 0"/>
     <axis xyz="0 0 1"/>
-    <limit lower="-0.785" upper="0.785" effort="100" velocity="1.0"/>
+    <limit lower="-0.4" upper="0.4" effort="100" velocity="1.0"/>
   </joint>
+  <xacro:system_steering_ros2_control update_rate="$(arg update_rate)"/>
 </robot>
